Commit message: astro raspberry: Updating aesthetics in urdf

File: raspberry_pi/src/astro_description/urdf/turtlebot3_burger_pi.urdf.xacro (robot description, xacro)
@@ -43,5 +43,5 @@
         <mesh filename="package://astro_description/meshes/wheels/left_tire.stl" scale="0.001 0.001 0.001"/>
       </geometry>
-      <material name="dark"/>
+      <material name="black"/>
     </visual>
     <collision>
@@ -71,5 +71,5 @@
         <mesh filename="package://astro_description/meshes/wheels/right_tire.stl" scale="0.001 0.001 0.001"/>
       </geometry>
-      <material name="dark"/>
+      <material name="black"/>
     </visual>
     <collision>
@@ -124,5 +124,5 @@
         <mesh filename="package://astro_description/meshes/sensors/lds.stl" scale="0.001 0.001 0.001"/>
       </geometry>
-      <material name="dark"/>
+      <material name="black"/>
     </visual>
     <collision>
