Commit message: Updating robot description to remove unnecessary files

File: ros2_ws/src/astro_robot_description/urdf/burger.urdf (robot description, URDF)
Before this commit: robot turtlebot3_burger, 7 links, 6 joints
Links:
- link base_link: geometry collision box size=0.140 0.140 0.143; visual mesh filename=package://turtlebot3_description/meshes/bases/burger_base.s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 scale=0.001 0.001 0.001
- link base_scan: geometry collision cylinder length=0.0315 radius=0.055; visual mesh filename=package://turtlebot3_description/meshes/sensors/lds.stl scale=0.001 0.001 0.001
- link wheel_left_link: geometry collision cylinder length=0.018 radius=0.033; visual mesh filename=package://turtlebot3_description/meshes/wheels/left_tire.stl scale=0.001 0.001 0.001
- link wheel_right_link: geometry collision cylinder length=0.018 radius=0.033; visual mesh filename=package://turtlebot3_description/meshes/wheels/right_tire.s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 scale=0.001 0.001 0.001

File: ros2_ws/src/astro_robot_description/urdf/waffle.urdf (robot description, URDF)
Before this commit: robot turtlebot3_waffle, 13 links, 12 joints
Links:
- link base_link: geometry collision box size=0.266 0.266 0.094; visual mesh filename=package://astro_robot_description/meshes/bases/waffle_base.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 scale=0.001 0.001 0.001
- link base_scan: geometry collision cylinder length=0.0315 radius=0.055; visual mesh filename=package://astro_robot_description/meshes/sensors/lds.stl scale=0.001 0.001 0.001
- link camera_link: geometry collision box size=0.012 0.132 0.020; visual mesh filename=package://astro_robot_description/meshes/sensors/r200.dae
- link wheel_left_link: geometry collision cylinder length=0.018 radius=0.033; visual mesh filename=package://astro_robot_description/meshes/wheels/left_tire.s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 scale=0.001 0.001 0.001
- link wheel_right_link: geometry collision cylinder length=0.018 radius=0.033; visual mesh filename=package://astro_robot_description/meshes/wheels/right_tire.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 scale=0.001 0.001 0.001
Joints:
- joint camera_depth_joint: origin xyz=${r200_cam_rgb_px} ${r200_cam_rgb_py + r200_cam_depth_offset} ${r200_cam_rgb_pz} rpy=0 0 0 -> xyz=0.005 0.028 0.013 rpy=0 0 0
- joint camera_rgb_joint: origin xyz=${r200_cam_rgb_px} ${r200_cam_rgb_py} ${r200_cam_rgb_pz} rpy=0 0 0 -> xyz=0.005 0.018 0.013 rpy=0 0 0
