Commit message: Issues Observed when running cartographer with TRAJECTORY_BUILDER_2D.use_imu_data = true
These were the issues I observed when setting TRAJECTORY_BUILDER_2D.use_imu_data = true

[cartographer logger]: W0215 23:00:25.000000 23436 tf_bridge.cpp:53] Invalid argument "" passed to lookupTransform argument source_frame - in tf2 frame_ids cannot be empty
This was fixed by adding the frame_id to the imu data in the astro_sensor node

[cartographer_node-1] F0215 23:10:29.476033 25356 sensor_bridge.cpp:136] Check failed: sensor_to_tracking->translation().norm() < 1e-5 The IMU frame must be colocated with the tracking frame. Transforming linear acceleration into the tracking frame will otherwise be imprecise. [cartographer_node-1] [FATAL] [1739682629.476279237] [cartographer logger]: F0215 23:10:29.000000 25356 sensor_bridge.cpp:136] Check failed: sensor_to_tracking->translation().norm() < 1e-5 The IMU frame must be colocated with the tracking frame. Transforming linear acceleration into the tracking frame will otherwise be imprecise.
Cartographer expects the IMU and tracking frame to be the same or very close.
This was fixed by making sure there is not rotational offset in the urdf file

[cartographer logger]: I0215 23:17:28.000000 26588 pose_graph_2d.cc:148] Inserted submap (0, 0). [cartographer_node-1] F0215 23:17:28.321084 26588 imu_tracker.cc:67] Check failed: (orientation_ * gravity_vector_).z() > 0. (0 vs. 0)  [cartographer_node-1] [FATAL] [1739683048.321357211] [cartographer logger]: F0215 23:17:28.000000 26588 imu_tracker.cc:67] Check failed: (orientation_ * gravity_vector_).z() > 0. (0 vs. 0)
Check failed: (orientation_ * gravity_vector_).z() > 0. suggests that Cartographer is failing because the IMU data is not correctly oriented with gravity. Essentially, Cartographer expects that when transformed, the gravity vector should point downward, but it's not, leading to a crash.
I observed that the I was not publishing any measurement data from the astro_sensor node after syncing it with time. This was fixed by copying the measurement data and pusblishing it after syncing with time
https://github.com/furhadjidda/astro/issues/3

File: ros2_ws/src/astro_robot_description/urdf/waffle.urdf (robot description, URDF)
Before this commit: robot turtlebot3_waffle, 13 links, 12 joints
Joints:
- joint imu_joint: origin xyz=0.0 0 0.068 rpy=0 0 0 -> xyz=0 0 0  rpy=0 0 0
